File: pcbs/keypads/keypadnew/keypadnew.kicad_pcb (KiCad board)
At the start: 2 copper layers, 60 x 40 mm, 17 parts, among them J1 Conn_01x02_Pin, J2 Conn_01x04_Pin, J3 Conn_01x02_Pin, J4 Conn_01x07_Pin, U1 ESP32-DEVKITC, U2 AMS1117-3.3, U3 AMS1117-3.3

Commit message: Update PCB Keypad Reader
Other:
- board text added: "FUELINX by Elefante"
Changed lines of the file:
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@@
   (gr_line (start 80.9 38.2) (end 80.9 72.2)
     (stroke (width 0.1) (type default)) (layer "Edge.Cuts"))
+  (gr_text "FUELINX\nby Elefante" (at 127.9 63.1) (layer "F.Cu")
+    (effects (font (size 1.5 1.5) (thickness 0.3) bold) (justify bottom))
+  )
+  (gr_text "FUELINX by Elefante" (at 122.5 51.6) (layer "B.Cu")
+    (effects (font (size 1.5 1.5) (thickness 0.3) bold) (justify left bottom mirror))
+  )
   (segment (start 121.5 54.8) (end 128.26 54.8) (width 1) (layer "F.Cu") (net 1))
   (segment (start 128.26 54.8) (end 134.98 48.08) (width 1) (layer "F.Cu") (net 1))

Commit message: Logo di PCB
Parts:
- added G***: LOGO, logo:fuellinx, F.Cu at (127.9, 58.4)
- added G***: LOGO, logo:fuellinx, B.Cu at (122.7, 48.0)
Other:
- board text added: "by Elefante"
- board text removed: "FUELINX by Elefante"
